Commit message: Added revtriplane files

File: PyFlyt/models/vehicles/revtriplane/revtriplane.urdf (robot description, URDF)
Before this commit: robot revtriplane, 10 links, 9 joints
Links:
- link ail_left_link: geometry collision box size=0.27 0.28 0.06; visual box size=0.27 0.28 0.06
- link ail_right_link: geometry collision box size=0.27 0.28 0.06; visual box size=0.27 0.28 0.06
- link base_link: mass 0.3 -> 0.4
- link front_motor_link: mass 0 -> 0.1
- link fuselage_link: mass 1 -> 0.8; geometry collision box size=1.0 0.05 0.05; visual box size=1.0 0.05 0.05
- link horizontal_tail_link: mass 0.1 -> 0.2
- link main_wing_link: mass 0.5 -> 1.0
- link vertical_tail_link: mass 0.05 -> 0.15; geometry collision box size=0.26 0.05 0.255; visual box size=0.26 0.05 0.255
Joints:
- joint ail_left_joint: origin xyz=-0.5 0.95 0 rpy=0 0 0 -> xyz=0.225 0.685 0 rpy=0 0 0
- joint ail_right_joint: origin xyz=-0.5 -0.95  0 rpy=0 0 0 -> xyz=0.225 -0.685  0 rpy=0 0 0
- joint fuselage_joint: origin xyz=-0.45 0 0 rpy=0 0 0 -> xyz=-0.15 0 0 rpy=0 0 0
- joint vertical_tail_joint: origin xyz=-0.65 0.0 0.0 rpy=0 0 0 -> xyz=-0.65 0.0 0.1275 rpy=0 0 0

Commit message: Updated triplane

File: PyFlyt/models/vehicles/revtriplane/revtriplane.urdf (robot description, URDF)
Before this commit: robot revtriplane, 10 links, 9 joints
Joints:
- joint front_motor_joint: origin xyz=0.57 0 0.1 rpy=0 0 0 -> xyz=0.57 0 0.0 rpy=0 0 0
- joint left_motor_joint: origin xyz=-0.19 0.405 0.1 rpy=0 0 0 -> xyz=-0.19 0.405 0.0 rpy=0 0 0
- joint right_motor_joint: origin xyz=-0.19 -0.405 0.1 rpy=0 0 0 -> xyz=-0.19 -0.405 0.0 rpy=0 0 0
